File: c14_rpi_svxlink_if.kicad_pcb (KiCad board)
At the start: 2 copper layers, 87 x 56 mm, 54 parts, among them J1 RPi_GPIO Tall, J2 Conn_01x04, J3 Conn_01x04, J4 Conn_01x04, J5 Conn_01x02, J6 Conn_01x04, J7 DB9F, Q1 BC847, Q2 BC847, Q3 BC847, Q4 BC857, Q5 BC847, T1 1:1, T2 1:1, U1 TLP222A o. AQY282EH, U2 HCPL-B17, U3 ADS1115_Module

Commit message: Neue Teile platziert, pre-1.1 bereit fuer Review
Parts:
- added C7: 1n, Capacitor_SMD:C_0805_2012Metric_Pad1.18x1.45mm_HandSolder, F.Cu at (194.9, 115.2)
- added C8: 1n, Capacitor_SMD:C_0805_2012Metric_Pad1.18x1.45mm_HandSolder, F.Cu at (199.3, 115.2)
- added D6: LL4148, Diode_SMD:D_MiniMELF, F.Cu at (197.4, 119.8)
- added D7: LL4148, Diode_SMD:D_MiniMELF, F.Cu at (195.1, 119.8)
- added FID1: Fiducial, Fiducial:Fiducial_1mm_Mask3mm, F.Cu at (131.0, 114.0)
- added FID2: Fiducial, Fiducial:Fiducial_1mm_Mask3mm, F.Cu at (209.9, 116.8)
- added FID3: Fiducial, Fiducial:Fiducial_1mm_Mask3mm, F.Cu at (198.6, 70.5)
- added J8: Conn_01x01_Male, Connector_PinHeader_2.54mm:PinHeader_1x01_P2.54mm_Vertical, F.Cu at (194.8, 71.0)
- added JP1: SolderJumper_2_Open, Jumper:SolderJumper-2_P1.3mm_Open_TrianglePad1.0x1.5mm, F.Cu at (153.2, 92.4)
- added JP2: SolderJumper_2_Open, Jumper:SolderJumper-2_P1.3mm_Open_TrianglePad1.0x1.5mm, F.Cu at (200.3, 119.7)
- added LOGO1: Logo_Open_Hardware_Small, Symbol:OSHW-Logo2_9.8x8mm_SilkScreen, F.Cu at (160.6, 117.7)
- added R20: 10k, Resistor_SMD:R_0805_2012Metric_Pad1.20x1.40mm_HandSolder, F.Cu at (149.8, 76.7)
- added TP1: Conn_01x09_Male, Connector_PinHeader_1.27mm:PinHeader_1x09_P1.27mm_Vertical, F.Cu at (200.5, 99.8)
- added TP2: Conn_01x03_Male, Connector_PinHeader_1.27mm:PinHeader_1x03_P1.27mm_Vertical, F.Cu at (207.3, 69.7)
- Q5: value BC847 -> IRLML0030
- R19: value 22k -> 1k
- moved Q5 16.7 mm to (149.3, 92.2)
- moved R15 12.5 mm to (184.4, 118.5), turned to 90 degrees
- moved R19 2.80 mm to (149.8, 74.8), turned to 180 degrees
Connections:
- J5 pad 1: Net-(D5-Pad1) -> Net-(J5-Pad1)
- J5 pad 3: Net-(J5-Pad3) -> Net-(D5-Pad1)
- Q5 pad 3: Net-(J5-Pad3) -> Net-(J5-Pad1)
Routing:
- net /TX_AUDIO+: track 12.9 -> 29.2 mm, vias 0 -> 1
- net /RX_AUDIO-: track 12.2 -> 27.3 mm, vias 0 -> 1
- net /SOUNDCARD_TX_AUDIO: track 52.2 -> 67.4 mm
- net Net-(Q5-Pad1): track 4.16 -> 19.0 mm
- net Net-(C5-Pad1): track 15.2 -> 3.31 mm
- net Net-(J5-Pad1): track 0.00 -> 10.6 mm
- net /RX_AUDIO+: track 19.5 -> 28.8 mm
- net Net-(J5-Pad3): track 8.74 -> 0.00 mm
- net GND: track 46.2 -> 38.1 mm
- net /TX_AUDIO-: track 45.4 -> 52.2 mm, vias 0 -> 1
- net /SOUNDCARD_RX_AUDIO: track 6.30 -> 11.9 mm
- net Net-(D6-Pad2): track 0.00 -> 5.52 mm
- net /RPI_FAN_TACHO: track 18.3 -> 15.2 mm
- net /RSSI: track 17.4 -> 20.3 mm, vias 0 -> 1
- net /SQL_DET-: track 79.3 -> 77.2 mm
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Other:
- board text added: "Jumper JP1 - Bypass PWM (always on) JP2 - Enable clipping diodes"
- board text added: "PWM"
- board text added: "R"
- board text added: "T"

Commit message: ready for production
Parts:
- added C9: 1n, Capacitor_SMD:C_0805_2012Metric_Pad1.18x1.45mm_HandSolder, F.Cu at (155.8, 92.4)
- added R21: 100R, Resistor_SMD:R_0805_2012Metric_Pad1.20x1.40mm_HandSolder, F.Cu at (203.7, 121.5)
- moved D6 1.25 mm to (196.4, 119.0)
- moved D7 1.25 mm to (194.1, 119.0)
- moved JP2 1.03 mm to (199.4, 120.2)
Connections:
- JP2 pad 1: Net-(D6-Pad2) -> Net-(JP2-Pad1)
Routing:
- net Net-(Q5-Pad1): track 19.0 -> 29.3 mm
- net Net-(JP2-Pad1): track 0.00 -> 5.91 mm
- net Net-(D6-Pad2): track 5.52 -> 9.14 mm
- net Net-(J5-Pad1): track 10.6 -> 14.0 mm, vias 0 -> 1
- net /RX_AUDIO+: track 28.8 -> 29.6 mm

Commit message: last changes for 1.1
Changed lines of the file:
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@@
       (layerselection 0x00010fc_ffffffff)
       (disableapertmacros false)
-      (usegerberextensions false)
-      (usegerberattributes true)
-      (usegerberadvancedattributes true)
-      (creategerberjobfile true)
+      (usegerberextensions true)
+      (usegerberattributes false)
+      (usegerberadvancedattributes false)
+      (creategerberjobfile false)
       (svguseinch false)
       (svgprecision 6)
@@
       (psa4output false)
       (plotreference true)
-      (plotvalue true)
+      (plotvalue false)
       (plotinvisibletext false)
       (sketchpadsonfab false)
-      (subtractmaskfromsilk false)
+      (subtractmaskfromsilk true)
       (outputformat 1)
       (mirror false)
-      (drillshape 1)
+      (drillshape 0)
       (scaleselection 1)
-      (outputdirectory "")
+      (outputdirectory "export/gerber")
     )
   )
@@
     (fp_line (start 1 0.625) (end -1 0.625) (layer "F.Fab") (width 0.1))
     (fp_line (start 1 -0.625) (end 1 0.625) (layer "F.Fab") (width 0.1))
-    (pad "1" smd roundrect (at -1 0 180) (size 1.2 1.4) (layers "F.Cu" "F.Paste" "F.Mask") (roundrect_rratio 0.208333)
+    (pad "1" smd roundrect (at -1 0 180) (size 1.2 1.4) (layers "F.Cu" "F.Paste" "F.Mask") (roundrect_rratio 0.2083333333)
       (net 22 "/RPI_FAN_CTRL") (pintype "passive"))
-    (pad "2" smd roundrect (at 1 0 180) (size 1.2 1.4) (layers "F.Cu" "F.Paste" "F.Mask") (roundrect_rratio 0.208333)
+    (pad "2" smd roundrect (at 1 0 180) (size 1.2 1.4) (layers "F.Cu" "F.Paste" "F.Mask") (roundrect_rratio 0.2083333333)
       (net 76 "Net-(Q5-Pad1)") (pintype "passive"))
     (model "${KICAD6_3DMODEL_DIR}/Resistor_SMD.3dshapes/R_0805_2012Metric.wrl"
@@
     (fp_line (start -1 -0.625) (end 1 -0.625) (layer "F.Fab") (width 0.1))
     (fp_line (start 1 -0.625) (end 1 0.625) (layer "F.Fab") (width 0.1))
-    (pad "1" smd roundrect (at -1.0375 0) (size 1.175 1.45) (layers "F.Cu" "F.Paste" "F.Mask") (roundrect_rratio 0.212766)
+    (pad "1" smd roundrect (at -1.0375 0) (size 1.175 1.45) (layers "F.Cu" "F.Paste" "F.Mask") (roundrect_rratio 0.2127659574)
       (net 46 "/RX_AUDIO-") (pintype "passive"))
-    (pad "2" smd roundrect (at 1.0375 0) (size 1.175 1.45) (layers "F.Cu" "F.Paste" "F.Mask") (roundrect_rratio 0.212766)
+    (pad "2" smd roundrect (at 1.0375 0) (size 1.175 1.45) (layers "F.Cu" "F.Paste" "F.Mask") (roundrect_rratio 0.2127659574)
       (net 47 "/RX_AUDIO+") (pintype "passive"))
     (model "${KICAD6_3DMODEL_DIR}/Capacitor_SMD.3dshapes/C_0805_2012Metric.wrl"
@@
     (fp_line (start -1 -0.625) (end 1 -0.625) (layer "F.Fab") (width 0.1))
     (fp_line (start 1 0.625) (end -1 0.625) (layer "F.Fab") (width 0.1))
-    (pad "1" smd roundrect (at -1.0375 0 90) (size 1.175 1.45) (layers "F.Cu" "F.Paste" "F.Mask") (roundrect_rratio 0.212766)
+    (pad "1" smd roundrect (at -1.0375 0 90) (size 1.175 1.45) (layers "F.Cu" "F.Paste" "F.Mask") (roundrect_rratio 0.2127659574)
       (net 1 "GND") (pintype "passive"))
-    (pad "2" smd roundrect (at 1.0375 0 90) (size 1.175 1.45) (layers "F.Cu" "F.Paste" "F.Mask") (roundrect_rratio 0.212766)
+    (pad "2" smd roundrect (at 1.0375 0 90) (size 1.175 1.45) (layers "F.Cu" "F.Paste" "F.Mask") (roundrect_rratio 0.2127659574)
       (net 76 "Net-(Q5-Pad1)") (pintype "passive"))
     (model "${KICAD6_3DMODEL_DIR}/Capacitor_SMD.3dshapes/C_0805_2012Metric.wrl"
@@
     (fp_line (start 1 -0.625) (end 1 0.625) (layer "F.Fab") (width 0.1))
     (fp_line (start -1 0.625) (end -1 -0.625) (layer "F.Fab") (width 0.1))
-    (pad "1" smd roundrect (at -1 0 180) (size 1.2 1.4) (layers "F.Cu" "F.Paste" "F.Mask") (roundrect_rratio 0.208333)
+    (pad "1" smd roundrect (at -1 0 180) (size 1.2 1.4) (layers "F.Cu" "F.Paste" "F.Mask") (roundrect_rratio 0.2083333333)
       (net 79 "Net-(JP2-Pad1)") (pintype "passive"))
-    (pad "2" smd roundrect (at 1 0 180) (size 1.2 1.4) (layers "F.Cu" "F.Paste" "F.Mask") (roundrect_rratio 0.208333)
+    (pad "2" smd roundrect (at 1 0 180) (size 1.2 1.4) (layers "F.Cu" "F.Paste" "F.Mask") (roundrect_rratio 0.2083333333)
       (net 78 "Net-(D6-Pad2)") (pintype "passive"))
     (model "${KICAD6_3DMODEL_DIR}/Resistor_SMD.3dshapes/R_0805_2012Metric.wrl"
@@
     (fp_line (start 7.45 3.4) (end 7.45 -2.35) (layer "F.Fab") (width 0.1))
     (fp_line (start -2.45 3.4) (end 7.45 3.4) (layer "F.Fab") (width 0.1))
-    (pad "1" thru_hole roundrect locked (at 0 0 90) (size 1.7 1.95) (drill 0.95) (layers *.Cu *.Mask) (roundrect_rratio 0.147059)
+    (pad "1" thru_hole roundrect locked (at 0 0 90) (size 1.7 1.95) (drill 0.95) (layers *.Cu *.Mask) (roundrect_rratio 0.1470588235)
       (net 77 "Net-(J5-Pad1)") (pinfunction "Pin_1") (pintype "passive"))
     (pad "2" thru_hole oval locked (at 2.5 0 90) (size 1.7 1.95) (drill 0.95) (layers *.Cu *.Mask)
@@
     (fp_line (start 1 -0.625) (end 1 0.625) (layer "F.Fab") (width 0.1))
     (fp_line (start -1 -0.625) (end 1 -0.625) (layer "F.Fab") (width 0.1))
-    (pad "1" smd roundrect (at -1 0 180) (size 1.2 1.4) (layers "F.Cu" "F.Paste" "F.Mask") (roundrect_rratio 0.208333)
+    (pad "1" smd roundrect (at -1 0 180) (size 1.2 1.4) (layers "F.Cu" "F.Paste" "F.Mask") (roundrect_rratio 0.2083333333)
       (net 22 "/RPI_FAN_CTRL") (pintype "passive"))
-    (pad "2" smd roundrect (at 1 0 180) (size 1.2 1.4) (layers "F.Cu" "F.Paste" "F.Mask") (roundrect_rratio 0.208333)
+    (pad "2" smd roundrect (at 1 0 180) (size 1.2 1.4) (layers "F.Cu" "F.Paste" "F.Mask") (roundrect_rratio 0.2083333333)
       (net 1 "GND") (pintype "passive"))
     (model "${KICAD6_3DMODEL_DIR}/Resistor_SMD.3dshapes/R_0805_2012Metric.wrl"
@@
     (fp_line (start 1 -0.625) (end 1 0.625) (layer "F.Fab") (width 0.1))
     (fp_line (start -1 -0.625) (end 1 -0.625) (layer "F.Fab") (width 0.1))
-    (pad "1" smd roundrect (at -1.0375 0 180) (size 1.175 1.45) (layers "F.Cu" "F.Paste" "F.Mask") (roundrect_rratio 0.212766)
+    (pad "1" smd roundrect (at -1.0375 0 180) (size 1.175 1.45) (layers "F.Cu" "F.Paste" "F.Mask") (roundrect_rratio 0.2127659574)
       (net 48 "/TX_AUDIO-") (pintype "passive"))
-    (pad "2" smd roundrect (at 1.0375 0 180) (size 1.175 1.45) (layers "F.Cu" "F.Paste" "F.Mask") (roundrect_rratio 0.212766)
+    (pad "2" smd roundrect (at 1.0375 0 180) (size 1.175 1.45) (layers "F.Cu" "F.Paste" "F.Mask") (roundrect_rratio 0.2127659574)
       (net 49 "/TX_AUDIO+") (pintype "passive"))
     (model "${KICAD6_3DMODEL_DIR}/Capacitor_SMD.3dshapes/C_0805_2012Metric.wrl"
