File: c14_rpi_svxlink_if.kicad_sch (KiCad schematic)
At the start: 52 parts, among them J1 RPi_GPIO, J2 Conn_01x04, J3 Conn_01x04, J4 Conn_01x04, J5 Conn_01x02, J6 Conn_01x04, J7 DB9F, Q1 BC847, Q2 BC847, Q3 BC847, Q4 BC857, T1 1:1, T2 1:1, U1 TLP222A, U2 HCPL-B17, U3 ADS1115_Module

Commit message: Small preproduction changes
Parts:
- C3: footprint Capacitor_THT:C_Rect_L7.2mm_W3.5mm_P5.00mm_FKS2_FKP2_MKS2_MKP2 -> Capacitor_THT:C_Rect_L7.2mm_W4.5mm_P5.00mm_FKS2_FKP2_MKS2_MKP2; PartNr_Mouser 871-B32529C1103M289 -> 871-B32529C105J189
- D1: PartNr_Mouser 755-SML-H12U8TT86C -> 755-SML-H12V8TT86C
- D3: value 18V -> TVS 18V; PartNr_Mouser 576-SMBJ18CA -> 494-SMBJ18CAE3/TR13
- J1: value RPi_GPIO -> RPi_GPIO Tall; PartNr_Mouser 485-2222 -> 485-1992
- R12, R18, R2, R7, R9: PartNr_Mouser 652-CR0805FX-1001EL -> 652-CR0805FX-1001ELF
- R13: PartNr_Mouser 652-CR0805FX-2201E -> 652-CR0805FX-2201ELF
- U1: value TLP222A -> TLP222A o. AQY282EH; PartNr_Mouser 757-TLP222AF -> AQY282EH
Connections:
- no-connect marks 31 -> 33
Changed lines of the file:
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@@
   (no_connect (at 238.76 74.93))
   (no_connect (at 238.76 77.47))
+  (no_connect (at 86.36 36.83))
+  (no_connect (at 86.36 39.37))
   (no_connect (at 238.76 69.85))
   (no_connect (at 86.36 44.45))
@@
       (effects (font (size 1.27 1.27)) hide)
     )
-    (property "PartNr_Mouser" "652-CR0805FX-1001EL" (id 4) (at 33.02 115.57 0)
+    (property "PartNr_Mouser" "652-CR0805FX-1001ELF" (id 4) (at 33.02 115.57 0)
       (effects (font (size 1.27 1.27)) hide)
     )
@@
       (effects (font (size 1.27 1.27)) hide)
     )
-    (property "PartNr_Mouser" "652-CR0805FX-2201E" (id 4) (at 149.86 158.75 0)
+    (property "PartNr_Mouser" "652-CR0805FX-2201ELF" (id 4) (at 149.86 158.75 0)
       (effects (font (size 1.27 1.27)) hide)
     )
@@
     (in_bom yes) (on_board yes) (fields_autoplaced)
     (property "Reference" "U1" (id 0) (at 74.93 92.5535 0))
-    (property "Value" "TLP222A" (id 1) (at 74.93 95.3286 0))
+    (property "Value" "TLP222A o. AQY282EH" (id 1) (at 74.93 95.3286 0))
     (property "Footprint" "Package_DIP:DIP-4_W7.62mm" (id 2) (at 69.85 105.41 0)
       (effects (font (size 1.27 1.27) italic) (justify left) hide)
@@
       (effects (font (size 1.27 1.27)) (justify left) hide)
     )
-    (property "PartNr_Mouser" "757-TLP222AF" (id 4) (at 74.93 100.33 0)
+    (property "PartNr_Mouser" "AQY282EH" (id 4) (at 74.93 100.33 0)
       (effects (font (size 1.27 1.27)) hide)
     )
@@
       (effects (font (size 1.524 1.524)))
     )
-    (property "Value" "RPi_GPIO" (id 1) (at 62.23 25.5451 0)
+    (property "Value" "RPi_GPIO Tall" (id 1) (at 62.23 25.5451 0)
       (effects (font (size 1.524 1.524)))
     )
@@
       (effects (font (size 1.524 1.524)))
     )
-    (property "PartNr_Mouser" "485-2222" (id 4) (at 43.18 29.21 0)
+    (property "PartNr_Mouser" "485-1992" (id 4) (at 43.18 29.21 0)
       (effects (font (size 1.27 1.27)) hide)
     )
@@
       (effects (font (size 1.27 1.27)) hide)
     )
-    (property "PartNr_Mouser" "755-SML-H12U8TT86C" (id 4) (at 33.02 124.46 0)
+    (property "PartNr_Mouser" "755-SML-H12V8TT86C" (id 4) (at 33.02 124.46 0)
       (effects (font (size 1.27 1.27)) hide)
     )
@@
     (property "Reference" "C3" (id 0) (at 143.51 73.8845 90))
     (property "Value" "1u" (id 1) (at 143.51 76.6596 90))
-    (property "Footprint" "Capacitor_THT:C_Rect_L7.2mm_W3.5mm_P5.00mm_FKS2_FKP2_MKS2_MKP2" (id 2) (at 139.7 80.9752 0)
+    (property "Footprint" "Capacitor_THT:C_Rect_L7.2mm_W4.5mm_P5.00mm_FKS2_FKP2_MKS2_MKP2" (id 2) (at 139.7 80.9752 0)
       (effects (font (size 1.27 1.27)) hide)
     )
@@
       (effects (font (size 1.27 1.27)) hide)
     )
-    (property "PartNr_Mouser" "871-B32529C1103M289" (id 4) (at 143.51 80.01 0)
+    (property "PartNr_Mouser" "871-B32529C105J189" (id 4) (at 143.51 80.01 0)
       (effects (font (size 1.27 1.27)) hide)
     )
@@
       (effects (font (size 1.27 1.27)) hide)
     )
-    (property "PartNr_Mouser" "652-CR0805FX-1001EL" (id 4) (at 223.52 72.39 0)
+    (property "PartNr_Mouser" "652-CR0805FX-1001ELF" (id 4) (at 223.52 72.39 0)
       (effects (font (size 1.27 1.27)) hide)
     )
@@
       (effects (font (size 1.27 1.27)) hide)
     )
-    (property "PartNr_Mouser" "652-CR0805FX-1001EL" (id 4) (at 62.23 153.67 0)
+    (property "PartNr_Mouser" "652-CR0805FX-1001ELF" (id 4) (at 62.23 153.67 0)
       (effects (font (size 1.27 1.27)) hide)
     )
@@
       (effects (font (size 1.27 1.27)) (justify right))
     )
-    (property "Value" "18V" (id 1) (at 88.392 102.1966 90)
+    (property "Value" "TVS 18V" (id 1) (at 88.392 102.1966 90)
       (effects (font (size 1.27 1.27)) (justify right))
     )
@@
       (effects (font (size 1.27 1.27)) hide)
     )
-    (property "PartNr_Mouser" "576-SMBJ18CA" (id 4) (at 86.36 100.33 0)
+    (property "PartNr_Mouser" "494-SMBJ18CAE3/TR13" (id 4) (at 86.36 100.33 0)
       (effects (font (size 1.27 1.27)) hide)
     )
@@
       (effects (font (size 1.27 1.27)) hide)
     )
-    (property "PartNr_Mouser" "652-CR0805FX-1001EL" (id 4) (at 76.2 172.72 0)
+    (property "PartNr_Mouser" "652-CR0805FX-1001ELF" (id 4) (at 76.2 172.72 0)
       (effects (font (size 1.27 1.27)) hide)
     )
@@
       (effects (font (size 1.27 1.27)) hide)
     )
-    (property "PartNr_Mouser" "652-CR0805FX-1001EL" (id 4) (at 106.68 161.29 0)
+    (property "PartNr_Mouser" "652-CR0805FX-1001ELF" (id 4) (at 106.68 161.29 0)
       (effects (font (size 1.27 1.27)) hide)
     )
@@
     )
     (path "/5ac81a20-d0be-4628-802b-923a0622c05a"
-      (reference "C3") (unit 1) (value "1u") (footprint "Capacitor_THT:C_Rect_L7.2mm_W3.5mm_P5.00mm_FKS2_FKP2_MKS2_MKP2")
+      (reference "C3") (unit 1) (value "1u") (footprint "Capacitor_THT:C_Rect_L7.2mm_W4.5mm_P5.00mm_FKS2_FKP2_MKS2_MKP2")
     )
     (path "/822f2848-7c51-4e15-8f68-690ddc412c7b"
@@
     )
     (path "/b56ad309-2a67-4ab5-a651-7cd4e5366e05"
-      (reference "D3") (unit 1) (value "18V") (footprint "Diode_SMD:D_SMA-SMB_Universal_Handsoldering")
+      (reference "D3") (unit 1) (value "TVS 18V") (footprint "Diode_SMD:D_SMA-SMB_Universal_Handsoldering")
     )
     (path "/900c5d1c-5597-4d7c-8021-a5d7fbabb7ea"
@@
     )
     (path "/38077e82-18b1-423c-84fa-424f895f4c90"
-      (reference "J1") (unit 1) (value "RPi_GPIO") (footprint "RPi_Hat:Pin_Header_Straight_2x20")
+      (reference "J1") (unit 1) (value "RPi_GPIO Tall") (footprint "RPi_Hat:Pin_Header_Straight_2x20")
     )
     (path "/22d31889-f524-400f-97ee-5171fa254853"
@@
     )
     (path "/343c38e1-c75e-4de0-9fc5-955497dd416c"
-      (reference "U1") (unit 1) (value "TLP222A") (footprint "Package_DIP:DIP-4_W7.62mm")
+      (reference "U1") (unit 1) (value "TLP222A o. AQY282EH") (footprint "Package_DIP:DIP-4_W7.62mm")
     )
     (path "/0024fded-4922-4bd8-a879-224d757e837b"

Commit message: Fix: Correct Footprint for J7 (M->F)
Parts:
- J7: footprint Connector_Dsub:DSUB-9_Male_Horizontal_P2.77x2.84mm_EdgePinOffset7.70mm_Housed_MountingHolesOffset9.12mm -> Connector_Dsub:DSUB-9_Female_Horizontal_P2.77x2.84mm_EdgePinOffset7.70mm_Housed_MountingHolesOffset9.12mm
Changed lines of the file:
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@@
       (effects (font (size 1.27 1.27)) (justify left))
     )
-    (property "Footprint" "Connector_Dsub:DSUB-9_Male_Horizontal_P2.77x2.84mm_EdgePinOffset7.70mm_Housed_MountingHolesOffset9.12mm" (id 2) (at 267.97 114.3 0)
+    (property "Footprint" "Connector_Dsub:DSUB-9_Female_Horizontal_P2.77x2.84mm_EdgePinOffset7.70mm_Housed_MountingHolesOffset9.12mm" (id 2) (at 267.97 114.3 0)
       (effects (font (size 1.27 1.27)) hide)
     )
@@
     )
     (path "/8ca3e20d-bcc7-4c5e-9deb-562dfed9fecb"
-      (reference "J7") (unit 1) (value "DB9F") (footprint "Connector_Dsub:DSUB-9_Male_Horizontal_P2.77x2.84mm_EdgePinOffset7.70mm_Housed_MountingHolesOffset9.12mm")
+      (reference "J7") (unit 1) (value "DB9F") (footprint "Connector_Dsub:DSUB-9_Female_Horizontal_P2.77x2.84mm_EdgePinOffset7.70mm_Housed_MountingHolesOffset9.12mm")
     )
     (path "/a3610b22-8fd5-480c-8522-b664b5b10a65"
